Commit message: removed unnecessary files

File: world_files/todo_copy_to_docker/to_copy_lidar/mp_400_with_lidar.urdf (robot description, URDF)
Before this commit: robot mp_400, 9 links, 8 joints
Links:
- added link lidar_2_link, mass 0.001; collision mesh filename=package://neo_simulation2/components/sensors/SICK-MICROSCAN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 scale=0.001 0.001 0.001; visual mesh filename=package://neo_simulation2/components/sensors/SICK-MICROSCAN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 scale=0.001 0.001 0.001
Joints:
- added joint lidar_1_joint: type fixed, parent base_link, child lidar_2_link, origin xyz=0.230 0 0.230 rpy=0 3.14 3.14, axis 0 0 1

Commit message: added instructions on adding lidar

File: world_files/todo_copy_to_docker/to_copy_lidar/mp_400_with_lidar.urdf (robot description, URDF)
Before this commit: robot mp_400, 10 links, 9 joints
Joints:
- joint lidar_1_joint: origin xyz=0.230 0 0.230 rpy=0 3.14 3.14 -> xyz=0.230 0 0.610 rpy=0 3.14 3.14
